File: frontEnd/gain.kicad_sch (KiCad schematic)
At the start: 14 parts, among them U501 MSA-0286, U502 BGS12P2L6E6327XTSA1, U503 BGS12P2L6E6327XTSA1

Commit message: update schematics, add bypass for the attenuator
Parts:
- added R505: 10, Resistor_SMD:R_0805_2012Metric, symbol Device:R_Small
- renumbered R503 to R504
Connections:
- net +12V: now also R505.1; no longer R504.1
- net at C505.2, C506.2, C507.2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: now also R505.2; no longer C503.1, U501.3 (RF_OUT)
- new net: C503.1, R504.1, U501.3 (RF_OUT)
Other:
- note added: "BIAS: 5V 40mA R504=(12-5)/0.040 R504=175 Gloss=20lg[(2*R504+50)/(2*R504)] Gloss=1.15db (because there's no RF choke following R504) GAIN=(-3+12-1.15) GAIN=7.85db"
- note removed: "BIAS: 5V 40mA R504=(12-5)/0.040 R504=175 Gloss=20lg[(2*R504+50)/(2*R504)] Gloss=1.15db GAIN=(-3+12-1.15) GAIN=7.85db"
- moved on the sheet: R504
Changed lines of the file:
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@@
   (junction (at 138.43 101.6) (diameter 0) (color 0 0 0 0)
   )
+  (junction (at 182.88 59.69) (diameter 0) (color 0 0 0 0)
+  )
   (junction (at 165.1 59.69) (diameter 0) (color 0 0 0 0)
   )
@@
     (stroke (width 0) (type default) (color 0 0 0 0))
   )
+  (wire (pts (xy 162.56 59.69) (xy 165.1 59.69))
+    (stroke (width 0) (type default) (color 0 0 0 0))
+  )
   (wire (pts (xy 80.01 105.41) (xy 80.01 106.68))
     (stroke (width 0) (type default) (color 0 0 0 0))
@@
     (stroke (width 0) (type default) (color 0 0 0 0))
   )
-  (wire (pts (xy 165.1 58.42) (xy 165.1 59.69))
-    (stroke (width 0) (type default) (color 0 0 0 0))
-  )
   (wire (pts (xy 210.82 85.09) (xy 210.82 86.36))
     (stroke (width 0) (type default) (color 0 0 0 0))
   )
+  (wire (pts (xy 154.94 59.69) (xy 157.48 59.69))
+    (stroke (width 0) (type default) (color 0 0 0 0))
+  )
   (wire (pts (xy 115.57 91.44) (xy 118.11 91.44))
     (stroke (width 0) (type default) (color 0 0 0 0))
@@
     (stroke (width 0) (type default) (color 0 0 0 0))
   )
-  (wire (pts (xy 165.1 52.07) (xy 165.1 53.34))
+  (wire (pts (xy 182.88 50.8) (xy 182.88 52.07))
     (stroke (width 0) (type default) (color 0 0 0 0))
   )
@@
     (stroke (width 0) (type default) (color 0 0 0 0))
   )
-  (wire (pts (xy 154.94 59.69) (xy 165.1 59.69))
-    (stroke (width 0) (type default) (color 0 0 0 0))
-  )
   (wire (pts (xy 165.1 59.69) (xy 173.99 59.69))
     (stroke (width 0) (type default) (color 0 0 0 0))
@@
     (stroke (width 0) (type default) (color 0 0 0 0))
   )
+  (wire (pts (xy 182.88 57.15) (xy 182.88 59.69))
+    (stroke (width 0) (type default) (color 0 0 0 0))
+  )
   (wire (pts (xy 167.64 91.44) (xy 201.93 91.44))
     (stroke (width 0) (type default) (color 0 0 0 0))
   )
-  (text "BIAS: 5V 40mA\nR504=(12-5)/0.040\nR504=175\nGloss=20lg[(2*R504+50)/(2*R504)]\nGloss=1.15db\nGAIN=(-3+12-1.15)\nGAIN=7.85db"
-    (at 121.92 63.5 0)
+  (text "BIAS: 5V 40mA\nR504=(12-5)/0.040\nR504=175\nGloss=20lg[(2*R504+50)/(2*R504)]\nGloss=1.15db (because there's no RF choke following R504)\nGAIN=(-3+12-1.15)\nGAIN=7.85db"
+    (at 177.8 180.34 0)
     (effects (font (size 1.27 1.27)) (justify left bottom))
   )
@@
     (pin "1")
   )
-  (symbol (lib_id "Device:R_Small") (at 165.1 55.88 0) (unit 1)
-    (in_bom yes) (on_board yes)
-    (property "Reference" "R503" (id 0) (at 166.37 54.61 0)
-      (effects (font (size 1.27 1.27)) (justify left))
-    )
-    (property "Value" "175" (id 1) (at 166.37 57.15 0)
-      (effects (font (size 1.27 1.27)) (justify left))
-    )
-    (property "Footprint" "Resistor_SMD:R_0805_2012Metric" (id 2) (at 165.1 55.88 0)
-      (effects (font (size 1.27 1.27)) hide)
-    )
-    (property "Datasheet" "~" (id 3) (at 165.1 55.88 0)
+  (symbol (lib_id "Device:R_Small") (at 160.02 59.69 90) (unit 1)
+    (in_bom yes) (on_board yes)
+    (property "Reference" "R504" (id 0) (at 158.75 58.42 0)
+      (effects (font (size 1.27 1.27)) (justify left))
+    )
+    (property "Value" "175" (id 1) (at 161.29 58.42 0)
+      (effects (font (size 1.27 1.27)) (justify left))
+    )
+    (property "Footprint" "Resistor_SMD:R_0805_2012Metric" (id 2) (at 160.02 59.69 0)
+      (effects (font (size 1.27 1.27)) hide)
+    )
+    (property "Datasheet" "~" (id 3) (at 160.02 59.69 0)
       (effects (font (size 1.27 1.27)) hide)
     )
@@
     (pin "1")
   )
-  (symbol (lib_id "power:+12V") (at 165.1 52.07 0) (unit 1)
-    (in_bom yes) (on_board yes)
-    (property "Reference" "#PWR?" (id 0) (at 165.1 55.88 0)
-      (effects (font (size 1.27 1.27)) hide)
-    )
-    (property "Value" "+12V" (id 1) (at 165.1 48.26 0))
-    (property "Footprint" "" (id 2) (at 165.1 52.07 0)
-      (effects (font (size 1.27 1.27)) hide)
-    )
-    (property "Datasheet" "" (id 3) (at 165.1 52.07 0)
+  (symbol (lib_id "Device:R_Small") (at 182.88 54.61 0) (unit 1)
+    (in_bom yes) (on_board yes)
+    (property "Reference" "R505" (id 0) (at 184.15 53.34 0)
+      (effects (font (size 1.27 1.27)) (justify left))
+    )
+    (property "Value" "10" (id 1) (at 184.15 55.88 0)
+      (effects (font (size 1.27 1.27)) (justify left))
+    )
+    (property "Footprint" "Resistor_SMD:R_0805_2012Metric" (id 2) (at 182.88 54.61 0)
+      (effects (font (size 1.27 1.27)) hide)
+    )
+    (property "Datasheet" "~" (id 3) (at 182.88 54.61 0)
+      (effects (font (size 1.27 1.27)) hide)
+    )
+    (pin "1")
+    (pin "2")
+  )
+  (symbol (lib_id "power:+12V") (at 182.88 50.8 0) (unit 1)
+    (in_bom yes) (on_board yes)
+    (property "Reference" "#PWR?" (id 0) (at 182.88 54.61 0)
+      (effects (font (size 1.27 1.27)) hide)
+    )
+    (property "Value" "+12V" (id 1) (at 182.88 46.99 0))
+    (property "Footprint" "" (id 2) (at 182.88 50.8 0)
+      (effects (font (size 1.27 1.27)) hide)
+    )
+    (property "Datasheet" "" (id 3) (at 182.88 50.8 0)
       (effects (font (size 1.27 1.27)) hide)
     )
@@
   )
   (symbol (lib_id "Device:C_Small") (at 173.99 63.5 180) (unit 1)
-    (in_bom yes) (on_board yes) (fields_autoplaced)
+    (in_bom yes) (on_board yes)
     (property "Reference" "C506" (id 0) (at 176.53 62.2235 0)
       (effects (font (size 1.27 1.27)) (justify right))
